File: KiCAD files/HS badge.kicad_pcb (KiCad board)
At the start: 2 copper layers, 55 x 69.8 mm, 21 parts, among them Q1 MMBT3906, Q2 MMBT3904, Q3 MMBT3904, Q4 MMBT3906, Q6 MMBT3904, SW1 SW_SPST

Commit message: Add files via upload
Parts:
- Q1, Q2, Q3, Q4, Q6: footprint Package_TO_SOT_SMD:SOT-23 -> Package_TO_SOT_SMD:TSOT-23_HandSoldering
- moved Q3 0.69 mm to (147.0, 93.3)
- moved Q1 0.30 mm to (153.7, 90.8)
Routing:
- net Net-(Q1-B): track 11.3 -> 12.9 mm
- net Net-(Q4-C): track 21.0 -> 22.3 mm
- net Net-(Q1-E): track 51.7 -> 50.7 mm
