File: KiCAD files/HS badge.kicad_sch (KiCad schematic)
At the start: 19 parts, among them Q1 MMBT3906, Q2 MMBT3904, Q3 MMBT3904, Q4 MMBT3906, Q6 MMBT3904, SW1 SW_SPST

Commit message: Add files via upload
Parts:
- Q1, Q2, Q3, Q4, Q6: footprint Package_TO_SOT_SMD:SOT-23 -> Package_TO_SOT_SMD:TSOT-23_HandSoldering
Changed lines of the file:
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@@
       (effects (font (size 1.27 1.27)) (justify left))
     )
-    (property "Footprint" "Package_TO_SOT_SMD:SOT-23" (at 160.02 94.615 0)
+    (property "Footprint" "Package_TO_SOT_SMD:TSOT-23_HandSoldering" (at 160.02 94.615 0)
       (effects (font (size 1.27 1.27) italic) (justify left) hide)
     )
@@
       (effects (font (size 1.27 1.27)) (justify left))
     )
-    (property "Footprint" "Package_TO_SOT_SMD:SOT-23" (at 134.62 127.635 0)
+    (property "Footprint" "Package_TO_SOT_SMD:TSOT-23_HandSoldering" (at 134.62 127.635 0)
       (effects (font (size 1.27 1.27) italic) (justify left) hide)
     )
@@
       (effects (font (size 1.27 1.27)) (justify left))
     )
-    (property "Footprint" "Package_TO_SOT_SMD:SOT-23" (at 201.93 84.455 0)
+    (property "Footprint" "Package_TO_SOT_SMD:TSOT-23_HandSoldering" (at 201.93 84.455 0)
       (effects (font (size 1.27 1.27) italic) (justify left) hide)
     )
@@
       (effects (font (size 1.27 1.27)) (justify left))
     )
-    (property "Footprint" "Package_TO_SOT_SMD:SOT-23" (at 181.61 84.455 0)
+    (property "Footprint" "Package_TO_SOT_SMD:TSOT-23_HandSoldering" (at 181.61 84.455 0)
       (effects (font (size 1.27 1.27) italic) (justify left) hide)
     )
@@
       (effects (font (size 1.27 1.27)) (justify left))
     )
-    (property "Footprint" "Package_TO_SOT_SMD:SOT-23" (at 173.99 104.775 0)
+    (property "Footprint" "Package_TO_SOT_SMD:TSOT-23_HandSoldering" (at 173.99 104.775 0)
       (effects (font (size 1.27 1.27) italic) (justify left) hide)
     )
